File: sensor-sch/EMGSensor2.2.sch (KiCad schematic (older format))
At the start: 22 parts, among them IC1 OPA1612, IC2 TL072

Commit message: fix R6 values in CAD files
Parts:
- R6: value 500Ω -> 100Ω
Changed lines of the file:
@@
 P 5188 4449
 F 0 "R6" V 5083 4492 50  0000 R CNN
-F 1 "500Ω" V 5275 4543 50  0000 R CNN
+F 1 "100Ω" V 5275 4543 50  0000 R CNN
 F 2 "" V 5228 4439 50  0001 C CNN
 F 3 "~" H 5188 4449 50  0001 C CNN
